File: Voyager60.kicad_pcb (KiCad board)
At the start: 2 copper layers, 285 x 95.1 mm, 265 parts, among them Q1 2N7002, SW1 5.2x5.2mm, U1 ATmega32U4-MU, U2 PRTR5V0U2X, Y1 16Mhz

Commit message: start changes
Parts:
- K_SPACE5: value MX-1.25U -> 2U; footprint MX_Alps_Hybrid:MX-1.25U-FLIPPED -> MX_Alps_Hybrid:MX-2U-ReversedStabilizers
- moved K_SPACE4 19.1 mm to (205.6, 108.0)
- moved K_SPACE5 11.9 mm to (160.3, 108.0)
- moved K_SPACE3 4.76 mm to (119.9, 108.0)
- moved R62 4.18 mm to (189.5, 113.5)
Routing:
- net LEDGND: track 1409.4 -> 1388.6 mm
- net +5V: track 1795.4 -> 1778.4 mm
- net COL6: track 369.3 -> 382.5 mm
- net Net-(K_SPACE4-Pad4): track 6.46 -> 19.1 mm
- net Net-(D62-Pad2): track 5.82 -> 18.0 mm
- net COL8: track 365.8 -> 375.5 mm
- net Net-(K_SPACE3-Pad4): track 6.46 -> 1.18 mm
- net COL4: track 243.6 -> 248.6 mm
- net Net-(D58-Pad2): track 5.82 -> 2.90 mm
- net Net-(K_SPACE1-Pad4): track 29.0 -> 30.5 mm
- net Net-(D61-Pad2): track 29.9 -> 30.6 mm
Other:
- net class Default removed
- net class Power removed

Commit message: start changing schematic
Parts:
- removed K_ALT1, K_CTRL1, K_RCTRL2, K_RWIN2, K_SHIFT2, K_WIN1: MX-1.25U, MX_Alps_Hybrid:MX-1.25U
- removed K_ENTER2: MX-ISO, MX_Alps_Hybrid:MX-ISO-ReversedStabilizers
- removed K_RALT2, K_RMENU2: MX-1.25U, MX_Alps_Hybrid:MX-1.25U-FLIPPED
- removed K_RSHIFT1: MX-2.75U, MX_Alps_Hybrid:MX-2.75U-FLIPPED
- removed K_SHIFT3, K_\2: MX-1U, MX_Alps_Hybrid:MX-1U
- removed K_SPACE1: MX-7U, MX_Alps_Hybrid:MX-7U-ReversedStabilizers
- removed K_SPACE2: MX-6.25U, MX_Alps_Hybrid:MX-6.25U-ReversedStabilizers
- K_#1, K_#10, K_#2, K_#3, K_#4, K_#5, K_#6, K_#7, K_#8, K_#9, K_'1, K_,1, K_-1, K_.1, K_/1, K_;1, K_=1, K_A1, K_B1, K_C1, K_D1, K_E1, K_ESC1, K_F1, K_G1, K_H1, K_I1, K_J1, K_K1, K_L1, K_M1, K_N1, K_O1, K_P1, K_Q1, K_R1, K_RWIN3, K_S1, K_SBACK1, K_SBACK2, K_SRSHIFT2, K_T1, K_U1, K_V1, K_W1, K_X1, K_Y1, K_Z1, K_[1, K_]1: value MX-1U -> 1U; footprint MX_Alps_Hybrid:MX-1U -> MX_Alps_Hybrid:MXOnly-1U-NoLED
- K_ALT2, K_CTRL2, K_RALT3, K_RCTRL3: footprint MX_Alps_Hybrid:MX-1.5U-FLIPPED -> MX_Alps_Hybrid:MXOnly-1.5U-NoLED
- K_BACK1: value MX-2U -> 2U; footprint MX_Alps_Hybrid:MX-2U -> MX_Alps_Hybrid:MXOnly-2U-NoLED
- K_CAPS1, K_SRSHIFT1: value MX-1.75U -> 1.75U; footprint MX_Alps_Hybrid:MX-1.75U -> MX_Alps_Hybrid:MXOnly-1.75U-NoLED
- K_CAPS2: footprint MX_Alps_Hybrid:MX-1.25U-FLIPPED -> MX_Alps_Hybrid:MXOnly-1.25U-NoLED
- K_ENTER1, K_SHIFT1: value MX-2.25U -> 2.25U; footprint MX_Alps_Hybrid:MX-2.25U -> MX_Alps_Hybrid:MXOnly-2.25U-NoLED
- K_SPACE3: footprint MX_Alps_Hybrid:MX-2.25U-ReversedStabilizers -> MX_Alps_Hybrid:MXOnly-2.25U-ReversedStabilizers-NoLED
- K_SPACE4: footprint MX_Alps_Hybrid:MX-2.75U-ReversedStabilizers -> MX_Alps_Hybrid:MXOnly-2.75U-ReversedStabilizers-NoLED
- K_SPACE5: footprint MX_Alps_Hybrid:MX-2U-ReversedStabilizers -> MX_Alps_Hybrid:MXOnly-2U-ReversedStabilizers-NoLED
- K_TAB1, K_\1: value MX-1.5U -> 1.5U; footprint MX_Alps_Hybrid:MX-1.5U -> MX_Alps_Hybrid:MXOnly-1.5U-NoLED
